Commit message: Chapter 2 version 1.0 upload

File: chapter_2/robot_description/urdf/pan_tilt.urdf (robot description, URDF)
Before this commit: robot pan_tilt, 4 links, 3 joints
Links:
- link base_link: geometry collision cylinder length=0.01 radius=0.2; visual cylinder length=0.01 radius=0.2
- link pan_link: geometry collision cylinder length=0.4 radius=0.04; visual cylinder length=0.4 radius=0.04
- link tilt_link: geometry collision cylinder length=0.4 radius=0.04; visual cylinder length=0.4 radius=0.04
Joints:
- removed joint world_fixed
- added joint world: type fixed, parent world, child base_link
